Commit message: still to get nodes running their own venvs, working on it

File: src/pi5_pkg/urdf/skid_steer_4wd.urdf (robot description, URDF)
Before this commit: robot skid_steer_4wd, 11 links, 10 joints
Links:
- link base_link: geometry collision box size=0.30 0.20 0.13; visual box size=0.25 0.13 0.005
- link cliff_front: geometry visual box size=0.04 0.015 0.005
- link cliff_rear: geometry visual box size=0.04 0.015 0.005
- link ld2450_front: geometry visual box size=0.005 0.015 0.05
- link sr04_rear: geometry visual box size=0.03 0.07 0.03
Joints:
- joint joint_camera_front: origin xyz=0.15 0 0.08 -> xyz=0.15 0 0.1
- joint joint_cliff_front: origin xyz=0.15 0.06 0.01 -> xyz=0.12 0.01 0.01
- joint joint_cliff_rear: origin xyz=-0.15 -0.06 0.01 -> xyz=-0.12 -0.01 0.01
- joint joint_ld2450_front: origin xyz=0.15 0 0.05 -> xyz=0.13 0 0.05
- joint joint_sr04_rear: origin xyz=-0.15 0 0.04 -> xyz=-0.13 0 0.04
- joint joint_vl53l5x_front: origin xyz=0.15 0 0.06 -> xyz=0.13 0 0.12
