Commit message: updated Readme.md

File: src/python_pkg/urdf/skid_steer_4wd.urdf (robot description, URDF)
Before this commit: robot skid_steer_4wd, 13 links, 12 joints
Links:
- removed link sr04_frt
- removed link sr04_rear
- added link front_sonar; visual box size=0.03 0.07 0.03
- added link rear_sonar; visual box size=0.03 0.07 0.03
Joints:
- joint joint_ld06: origin xyz=0.02 0.0 0.18 rpy=0 0 1.5708 -> xyz=0.02 0.0 0.18 rpy=0 0 -1.5708
- joint joint_sr04_front: child sr04_frt -> front_sonar; origin xyz=0.13 0 0.04 -> xyz=0.13 0 0.04 rpy=0 0 0
- joint joint_sr04_rear: child sr04_rear -> rear_sonar; origin xyz=-0.13 0 0.04 -> xyz=-0.13 0 0.04 rpy=0 0 3.14159
