Commit message: 1. Fixed errors in urdfs that were causing orientation of ld06 map by 90 degrees. 2. fixed main.cpp to detect gyro bias at start. unfortunately still retains around 0.005 radians bias. This needs a new logic in future to continually check and correct gyro bias. 3. Updated readme.md to set the template a bit better. 4. Renamed packages 5. updated hw_mcu_node.py to correct indentation. 6. added a main repo requirements.txt file.  7. portnames for UART-to-USB updated to the immutable names rather than /dev/ttyTHS1 etc. 8. added jetsoncpp launch file.  9. Fleshed out definition of isaac  launchfile.

File: src/jetsoncpp_pkg/urdf/skid_steer_4wd.urdf (robot description, URDF)
Before this commit: robot skid_steer_4wd, 13 links, 12 joints
Links:
- removed link sr04_frt
- removed link sr04_rear
- added link front_sonar; visual box size=0.03 0.07 0.03
- added link rear_sonar; visual box size=0.03 0.07 0.03
Joints:
- joint joint_ld06: origin xyz=0.02 0.0 0.18 -> xyz=0.02 0.0 0.18 rpy=0 0 -1.5708
- joint joint_sr04_front: child sr04_frt -> front_sonar; origin xyz=0.13 0 0.04 -> xyz=0.13 0 0.04 rpy=0 0 0
- joint joint_sr04_rear: child sr04_rear -> rear_sonar; origin xyz=-0.13 0 0.04 -> xyz=-0.13 0 0.04 rpy=0 0 3.14159

File: src/python_pkg/urdf/skid_steer_4wd.urdf (robot description, URDF)
Before this commit: robot skid_steer_4wd, 13 links, 12 joints
Joints:
- joint joint_ld06: origin xyz=0.02 0.0 0.18 -> xyz=0.02 0.0 0.18 rpy=0 0 1.5708

Commit message: Summary of Changes    1. hw_mcu_node.cpp Enhancements:        * Sensor Covariance: Added realistic covariance matrices to IMU and Odometry messages. This tells the EKF how much to "trust" the wheel encoders vs. the VSLAM data.        * Topic Namespacing: Renamed the raw MCU odometry to /mcu/odom to distinguish it from the fused /odom output.        * TF Toggle: Added an enable_tf_broadcast parameter, which I've disabled in the new launch file to allow the EKF to own the odom → base_link transform.    2. EKF Configuration (src/jetsoncpp_pkg/config/ekf.yaml):        * Fuses Wheel Odometry (Linear X), IMU (Angular Z / Yaw), and cuVSLAM (Pose X, Y, Yaw and Linear X).        * This provides a smooth, high-frequency odometry source that remains robust even if the camera is momentarily obscured.    3. Unified Launch File (src/jetsoncpp_pkg/launch/full_system.launch.py):        * Isaac ROS VSLAM: Configured to provide tracking data without publishing its own map or odom transforms, acting as a sensor input for the EKF.        * SLAM Toolbox: Consumes the LD06 Lidar data and the fused EKF odometry to perform mapping and provide the global map → odom correction.        * MCU & Lidar: Automatically initializes the serial communication and the Lidar PWM control.   How to Run   After building your workspace (colcon build --packages-select jetsoncpp_pkg), you can launch the entire fused system with:    1 ros2 launch jetsoncpp_pkg full_system.launch.py   This setup will provide a robust navigation stack where the Lidar corrects the VSLAM drift, and the Wheel Odometry stabilizes the VSLAM tracking.

File: src/jetsoncpp_pkg/urdf/skid_steer_4wd.urdf (robot description, URDF)
Before this commit: robot skid_steer_4wd, 13 links, 12 joints
Links:
- added link camera_depth_frame
- added link camera_depth_optical_frame
- added link camera_infra1_frame
- added link camera_infra1_optical_frame
- added link camera_infra2_frame
- added link camera_infra2_optical_frame
- added link camera_link
Joints:
- added joint joint_camera_depth_frame: type fixed, parent camera_link, child camera_depth_frame, origin xyz=0 0 0 rpy=0 0 0
- added joint joint_camera_depth_optical_frame: type fixed, parent camera_depth_frame, child camera_depth_optical_frame, origin xyz=0 0 0 rpy=-1.5708 0 -1.5708
- added joint joint_camera_infra1_frame: type fixed, parent camera_link, child camera_infra1_frame, origin xyz=0 0 0 rpy=0 0 0
- added joint joint_camera_infra1_optical_frame: type fixed, parent camera_infra1_frame, child camera_infra1_optical_frame, origin xyz=0 0 0 rpy=-1.5708 0 -1.5708
- added joint joint_camera_infra2_frame: type fixed, parent camera_link, child camera_infra2_frame, origin xyz=0 0 0 rpy=0 0 0
- added joint joint_camera_infra2_optical_frame: type fixed, parent camera_infra2_frame, child camera_infra2_optical_frame, origin xyz=0 0 0 rpy=-1.5708 0 -1.5708
- added joint joint_camera_link: type fixed, parent camera_binoc, child camera_link, origin xyz=0 0 0 rpy=0 0 0

Commit message: feat: implement sim_mcu_node and migrate to ros2_control for Gazebo simulation compatibility

File: src/jetsoncpp_pkg/urdf/skid_steer_4wd.urdf (robot description, URDF)
Before this commit: robot skid_steer_4wd, 20 links, 19 joints
Links:
- added link imu_link; visual box size=0.02 0.02 0.01
Joints:
- added joint joint_imu: type fixed, parent base_link, child imu_link, origin xyz=0 0.1 0.01 rpy=0 0 0

File: src/jetsoncpp_pkg/urdf/skid_steer_4wd_sim.urdf (robot description, URDF)
Before this commit: robot skid_steer_4wd_sim, 8 links, 7 joints
Links:
- added link imu_link, mass 0.01
Joints:
- added joint joint_imu: type fixed, parent base_link, child imu_link, origin xyz=0 0.1 0.01 rpy=0 0 0
