Commit message: updated setup-env to set shortcut commands.  Updated sim_mcu_node and hw_mcu_node to set correct cae conventions. checked that hw_mcu_node still works for manual driving. gazebo.launch is changed to use new gazebo.  need to verify gazebo.,launch and nav_sim.launch later

File: src/jetsoncpp_pkg/urdf/skid_steer_4wd_sim.urdf (robot description, URDF)
Before this commit: robot skid_steer_4wd_sim, 9 links, 8 joints
Links:
- removed link camera_depth_optical_frame
- removed link camera_link_sim
- added link camera_binoc; visual box size=0.025 0.10 0.02
- added link front_sonar; visual box size=0.03 0.07 0.03
- added link rear_sonar; visual box size=0.03 0.07 0.03
- link base_link: mass 5.0 -> 2.0; geometry collision box size=0.25 0.13 0.05; visual box size=0.25 0.13 0.004
- link imu_link: geometry visual box size=0.02 0.02 0.01
- link ld06_lidar: geometry visual cylinder length=0.015 radius=0.02
Joints:
- removed joint joint_camera_sim
- removed joint joint_depth_optical
- added joint joint_camera_binoc: type fixed, parent base_link, child camera_binoc, origin xyz=0.06 -0.01 0.13
- added joint joint_sr04_front: type fixed, parent base_link, child front_sonar, origin xyz=0.13 0 0.04
- added joint joint_sr04_rear: type fixed, parent base_link, child rear_sonar, origin xyz=-0.13 0 0.04 rpy=0 0 3.14159
- joint joint_ld06: origin xyz=0.02 0.0 0.18 rpy=0 0 0 -> xyz=0.02 0.0 0.18 rpy=0 0 -1.5708
