Commit message: refactor: update wheel collision geometry and migrate gazebo plugins to ignition counterparts

File: src/jetcar_description/urdf/jetcar.urdf.xacro (robot description, xacro)
@@ -36,6 +36,6 @@
       </visual>
       <collision>
-        <geometry><cylinder length="0.03" radius="0.035"/></geometry>
-        <origin xyz="0 0 0" rpy="1.5708 0 0"/>
+        <geometry><sphere radius="0.035"/></geometry>
+        <origin xyz="0 0 0" rpy="0 0 0"/>
       </collision>
       <inertial>
@@ -96,5 +96,5 @@
   <xacro:if value="$(arg sim_mode)">
     <ros2_control name="GazeboSimSystem" type="system">
-      <hardware><plugin>gz_ros2_control/GazeboSimSystem</plugin></hardware>
+      <hardware><plugin>ign_ros2_control/IgnitionSystem</plugin></hardware>
       <joint name="joint_wheel_fl"><command_interface name="effort"/><state_interface name="position"/><state_interface name="velocity"/><state_interface name="effort"/></joint>
       <joint name="joint_wheel_fr"><command_interface name="effort"/><state_interface name="position"/><state_interface name="velocity"/><state_interface name="effort"/></joint>
@@ -103,8 +103,8 @@
     </ros2_control>
     <gazebo>
-      <plugin filename="gz_ros2_control-system" name="gz_ros2_control::GazeboSimROS2ControlSystem">
+      <plugin filename="ign_ros2_control-system" name="ign_ros2_control::IgnitionROS2ControlPlugin">
         <parameters>$(find jetcar_sim)/config/sim_controllers.yaml</parameters>
       </plugin>
-      <plugin filename="gz-sim-odometry-publisher-system" name="gz::sim::systems::OdometryPublisher">
+      <plugin filename="libignition-gazebo-odometry-publisher-system.so" name="ignition::gazebo::systems::OdometryPublisher">
         <odom_frame>odom</odom_frame>
         <robot_base_frame>base_link</robot_base_frame>

Commit message: fix: adjust vertical offsets for camera, lidar, and imu joints in urdf model

File: src/jetcar_description/urdf/jetcar.urdf.xacro (robot description, xacro)
@@ -67,5 +67,5 @@
   <!-- Camera -->
   <link name="camera_binoc"><visual><geometry><box size="0.025 0.10 0.02"/></geometry><origin xyz="0 0 0.06"/><material name="green"/></visual></link>
-  <joint name="joint_camera_binoc" type="fixed"><parent link="base_link"/><child link="camera_binoc"/><origin xyz="0.06 -0.01 0.13"/></joint>
+  <joint name="joint_camera_binoc" type="fixed"><parent link="base_link"/><child link="camera_binoc"/><origin xyz="0.06 -0.01 0.145"/></joint>
   <link name="camera_link"/>
   <joint name="joint_camera_link" type="fixed"><parent link="camera_binoc"/><child link="camera_link"/><origin xyz="0 0 0"/></joint>
@@ -85,7 +85,7 @@
   <!-- Lidar & Other Sensors -->
   <link name="ld06_lidar"><visual><geometry><cylinder length="0.015" radius="0.02"/></geometry><material name="purple"/></visual><inertial><mass value="0.1"/><inertia ixx="0.001" ixy="0" ixz="0" iyy="0.001" iyz="0" izz="0.001"/></inertial></link>
-  <joint name="joint_ld06" type="fixed"><parent link="base_link"/><child link="ld06_lidar"/><origin xyz="0.02 0.0 0.18" rpy="0 0 -1.5708"/></joint>
+  <joint name="joint_ld06" type="fixed"><parent link="base_link"/><child link="ld06_lidar"/><origin xyz="0.02 0.0 0.24" rpy="0 0 -1.5708"/></joint>
   <link name="imu_link"><visual><geometry><box size="0.02 0.02 0.01"/></geometry><material name="blue"/></visual><inertial><mass value="0.01"/><inertia ixx="0.0001" ixy="0" ixz="0" iyy="0.0001" iyz="0" izz="0.0001"/></inertial></link>
-  <joint name="joint_imu" type="fixed"><parent link="base_link"/><child link="imu_link"/><origin xyz="0 0.1 0.01"/></joint>
+  <joint name="joint_imu" type="fixed"><parent link="base_link"/><child link="imu_link"/><origin xyz="0.0 0.07 0.07"/></joint>
   <!-- ToF & Radar (Visuals only) -->
   <link name="vl53l5x_front"><visual><geometry><box size="0.01 0.02 0.01"/></geometry><origin xyz="0 0 0.06"/><material name="yellow"/></visual></link>

Commit message: feat: migrate transform broadcasting to Gazebo bridge and refine sensor joint offsets

File: src/jetcar_description/urdf/jetcar.urdf.xacro (robot description, xacro)
@@ -67,5 +67,5 @@
   <!-- Camera -->
   <link name="camera_binoc"><visual><geometry><box size="0.025 0.10 0.02"/></geometry><origin xyz="0 0 0.06"/><material name="green"/></visual></link>
-  <joint name="joint_camera_binoc" type="fixed"><parent link="base_link"/><child link="camera_binoc"/><origin xyz="0.06 -0.01 0.145"/></joint>
+  <joint name="joint_camera_binoc" type="fixed"><parent link="base_link"/><child link="camera_binoc"/><origin xyz="0.06 -0.01 0.13"/></joint>
   <link name="camera_link"/>
   <joint name="joint_camera_link" type="fixed"><parent link="camera_binoc"/><child link="camera_link"/><origin xyz="0 0 0"/></joint>
@@ -85,7 +85,7 @@
   <!-- Lidar & Other Sensors -->
   <link name="ld06_lidar"><visual><geometry><cylinder length="0.015" radius="0.02"/></geometry><material name="purple"/></visual><inertial><mass value="0.1"/><inertia ixx="0.001" ixy="0" ixz="0" iyy="0.001" iyz="0" izz="0.001"/></inertial></link>
-  <joint name="joint_ld06" type="fixed"><parent link="base_link"/><child link="ld06_lidar"/><origin xyz="0.02 0.0 0.24" rpy="0 0 -1.5708"/></joint>
+  <joint name="joint_ld06" type="fixed"><parent link="base_link"/><child link="ld06_lidar"/><origin xyz="0.02 0.0 0.18" rpy="0 0 -1.5708"/></joint>
   <link name="imu_link"><visual><geometry><box size="0.02 0.02 0.01"/></geometry><material name="blue"/></visual><inertial><mass value="0.01"/><inertia ixx="0.0001" ixy="0" ixz="0" iyy="0.0001" iyz="0" izz="0.0001"/></inertial></link>
-  <joint name="joint_imu" type="fixed"><parent link="base_link"/><child link="imu_link"/><origin xyz="0.0 0.07 0.07"/></joint>
+  <joint name="joint_imu" type="fixed"><parent link="base_link"/><child link="imu_link"/><origin xyz="0 0.1 0.01"/></joint>
   <!-- ToF & Radar (Visuals only) -->
   <link name="vl53l5x_front"><visual><geometry><box size="0.01 0.02 0.01"/></geometry><origin xyz="0 0 0.06"/><material name="yellow"/></visual></link>

Commit message: Updated sim_robot system to have correct imu  topic.  integrate binocular infrared cameras in urdf.  updated navigation parameters and launch configuration

File: src/jetcar_description/urdf/jetcar.urdf.xacro (robot description, xacro)
@@ -67,5 +67,5 @@
   <!-- Camera -->
   <link name="camera_binoc"><visual><geometry><box size="0.025 0.10 0.02"/></geometry><origin xyz="0 0 0.06"/><material name="green"/></visual></link>
-  <joint name="joint_camera_binoc" type="fixed"><parent link="base_link"/><child link="camera_binoc"/><origin xyz="0.06 -0.01 0.13"/></joint>
+  <joint name="joint_camera_binoc" type="fixed"><parent link="base_link"/><child link="camera_binoc"/><origin xyz="0.06 -0.01 0.18"/></joint>
   <link name="camera_link"/>
   <joint name="joint_camera_link" type="fixed"><parent link="camera_binoc"/><child link="camera_link"/><origin xyz="0 0 0"/></joint>
@@ -76,16 +76,16 @@
   <joint name="joint_camera_depth_optical_frame" type="fixed"><parent link="camera_depth_frame"/><child link="camera_depth_optical_frame"/><origin xyz="0 0 0" rpy="-1.5708 0 -1.5708"/></joint>
   <link name="camera_infra1_frame"/>
-  <joint name="joint_camera_infra1_frame" type="fixed"><parent link="camera_link"/><child link="camera_infra1_frame"/><origin xyz="0 0 0"/></joint>
+  <joint name="joint_camera_infra1_frame" type="fixed"><parent link="camera_link"/><child link="camera_infra1_frame"/><origin xyz="0 0.025 0"/></joint>
   <link name="camera_infra1_optical_frame"/>
   <joint name="joint_camera_infra1_optical_frame" type="fixed"><parent link="camera_infra1_frame"/><child link="camera_infra1_optical_frame"/><origin xyz="0 0 0" rpy="-1.5708 0 -1.5708"/></joint>
   <link name="camera_infra2_frame"/>
-  <joint name="joint_camera_infra2_frame" type="fixed"><parent link="camera_link"/><child link="camera_infra2_frame"/><origin xyz="0 0 0"/></joint>
+  <joint name="joint_camera_infra2_frame" type="fixed"><parent link="camera_link"/><child link="camera_infra2_frame"/><origin xyz="0 -0.025 0"/></joint>
   <link name="camera_infra2_optical_frame"/>
   <joint name="joint_camera_infra2_optical_frame" type="fixed"><parent link="camera_infra2_frame"/><child link="camera_infra2_optical_frame"/><origin xyz="0 0 0" rpy="-1.5708 0 -1.5708"/></joint>
   <!-- Lidar & Other Sensors -->
   <link name="ld06_lidar"><visual><geometry><cylinder length="0.015" radius="0.02"/></geometry><material name="purple"/></visual><inertial><mass value="0.1"/><inertia ixx="0.001" ixy="0" ixz="0" iyy="0.001" iyz="0" izz="0.001"/></inertial></link>
-  <joint name="joint_ld06" type="fixed"><parent link="base_link"/><child link="ld06_lidar"/><origin xyz="0.02 0.0 0.18" rpy="0 0 -1.5708"/></joint>
+  <joint name="joint_ld06" type="fixed"><parent link="base_link"/><child link="ld06_lidar"/><origin xyz="0.02 0.0 0.22" rpy="0 0 -1.5708"/></joint>
   <link name="imu_link"><visual><geometry><box size="0.02 0.02 0.01"/></geometry><material name="blue"/></visual><inertial><mass value="0.01"/><inertia ixx="0.0001" ixy="0" ixz="0" iyy="0.0001" iyz="0" izz="0.0001"/></inertial></link>
-  <joint name="joint_imu" type="fixed"><parent link="base_link"/><child link="imu_link"/><origin xyz="0 0.1 0.01"/></joint>
+  <joint name="joint_imu" type="fixed"><parent link="base_link"/><child link="imu_link"/><origin xyz="0 0.1 0.07"/></joint>
   <!-- ToF & Radar (Visuals only) -->
   <link name="vl53l5x_front"><visual><geometry><box size="0.01 0.02 0.01"/></geometry><origin xyz="0 0 0.06"/><material name="yellow"/></visual></link>
@@ -123,4 +123,28 @@
       </sensor>
     </gazebo>
+    <!-- Left IR (Infra1) -->
+    <gazebo reference="camera_infra1_frame">
+      <sensor name="camera_infra1" type="camera">
+        <gz_frame_id>camera_infra1_frame</gz_frame_id>
+        <update_rate>15</update_rate>
+        <camera>
+          <horizontal_fov>1.204</horizontal_fov>
+          <image><width>640</width><height>480</height><format>L8</format></image>
+          <clip><near>0.1</near><far>10.0</far></clip>
+        </camera>
+      </sensor>
+    </gazebo>
+    <!-- Right IR (Infra2) -->
+    <gazebo reference="camera_infra2_frame">
+      <sensor name="camera_infra2" type="camera">
+        <gz_frame_id>camera_infra2_frame</gz_frame_id>
+        <update_rate>15</update_rate>
+        <camera>
+          <horizontal_fov>1.204</horizontal_fov>
+          <image><width>640</width><height>480</height><format>L8</format></image>
+          <clip><near>0.1</near><far>10.0</far></clip>
+        </camera>
+      </sensor>
+    </gazebo>
     <gazebo reference="ld06_lidar">
       <sensor name="ld06_lidar" type="gpu_lidar">

Commit message: chore: optimize camera resolution to 424x240, increase simulation motor torque, and refine wheel friction models to avoid slipping during turns.

File: src/jetcar_description/urdf/jetcar.urdf.xacro (robot description, xacro)
@@ -134,5 +134,5 @@
         <camera>
           <horizontal_fov>1.204</horizontal_fov>
-          <image><width>640</width><height>480</height><format>L8</format></image>
+          <image><width>424</width><height>240</height><format>L8</format></image>
           <clip><near>0.1</near><far>10.0</far></clip>
         </camera>
@@ -148,5 +148,5 @@
         <camera>
           <horizontal_fov>1.204</horizontal_fov>
-          <image><width>640</width><height>480</height><format>L8</format></image>
+          <image><width>424</width><height>240</height><format>L8</format></image>
           <clip><near>0.1</near><far>10.0</far></clip>
         </camera>
@@ -173,8 +173,8 @@
       </sensor>
     </gazebo>
-    <gazebo reference="wheel_fl"><mu>1.0</mu><mu2>1.0</mu2></gazebo>
-    <gazebo reference="wheel_fr"><mu>1.0</mu><mu2>1.0</mu2></gazebo>
-    <gazebo reference="wheel_rl"><mu>1.0</mu><mu2>1.0</mu2></gazebo>
-    <gazebo reference="wheel_rr"><mu>1.0</mu><mu2>1.0</mu2></gazebo>
+    <gazebo reference="wheel_fl"><collision><surface><friction><ode><mu>1.0</mu><mu2>1.0</mu2><fdir1>1 0 0</fdir1></ode></friction></surface></collision></gazebo>
+    <gazebo reference="wheel_fr"><collision><surface><friction><ode><mu>1.0</mu><mu2>1.0</mu2><fdir1>1 0 0</fdir1></ode></friction></surface></collision></gazebo>
+    <gazebo reference="wheel_rl"><collision><surface><friction><ode><mu>1.0</mu><mu2>1.0</mu2><fdir1>1 0 0</fdir1></ode></friction></surface></collision></gazebo>
+    <gazebo reference="wheel_rr"><collision><surface><friction><ode><mu>1.0</mu><mu2>1.0</mu2><fdir1>1 0 0</fdir1></ode></friction></surface></collision></gazebo>
   </xacro:if>
 </robot>

Commit message: feat: add wheel joint dynamics and tighten controller command timeout thresholds to avoid issue of '1 button press and it drives until hitting wall'

File: src/jetcar_description/urdf/jetcar.urdf.xacro (robot description, xacro)
@@ -49,4 +49,5 @@
       <origin xyz="${x} ${y} 0.035" rpy="0 0 0"/>
       <axis xyz="0 1 0"/>
+      <dynamics damping="0.5" friction="0.2"/>
     </joint>
   </xacro:macro>

Commit message: tuned friction and timeout  to try move it faster

File: src/jetcar_description/urdf/jetcar.urdf.xacro (robot description, xacro)
@@ -49,5 +49,5 @@
       <origin xyz="${x} ${y} 0.035" rpy="0 0 0"/>
       <axis xyz="0 1 0"/>
-      <dynamics damping="0.5" friction="0.2"/>
+      <dynamics damping="0.3" friction="0.1"/>
     </joint>
   </xacro:macro>
